File: MotorSystemVS1/Motorsystem.brd (EAGLE design)
At the start: 80 x 50 mm, 3 parts

Commit message: continue
Parts:
- removed BOX10P-L1: BOX10PBOX10P-T, connectors:BOX10P-T
- added CC1, CC2: 0.1u, capacitor:C1608
- added CN1: BOX10P-T, connectors:BOX10P-T
- added IC1: MCP2562-SN, Microchip:SOIC8
- added MCU1: NUCLEO-F303K8, Nucleo:NUCLEO-NANO
- added SW1: KHS42SMD, switch:KHS42
- added U$3: DF1B_L_4P, user:DF1B_L_4P
- added U$4, U$6, U$7, U$8: NP52N06SLG, user:NP52N06SLG
- added U$5: A3921, user:A3921
- added U$9: VL_4P, user:VL_4P
- U$1: value NUCLEO-F303K8 -> TLP2395; device Nucleo:NUCLEO-NANO -> user:TLP2395
- U$2: value MCP2561MCP2561-SN -> SOT23_NFET; device Microchip:SOIC8 -> user:SOT23_NFET
- moved U$2 29.0 mm to (34.3, 38.1), turned to 90 degrees
- moved U$1 12.0 mm to (33.0, 29.2), flipped to the bottom, turned to 180 degrees
Connections:
- new net CS: MCU1.P$19
- new net ENC_A: MCU1.P$23
- new net ENC_B: MCU1.P$20
- new net GND_MS: U$5.PAD, U$5.PIN17
- new net N$1: U$1.K, U$2.PIN3_D
- new net PWM: MCU1.P$12, U$2.PIN1_G
- new net PWM_MS: U$1.OUT, U$5.PIN22
- new net SW0: MCU1.P$15, SW1.P$8
- new net SW1: MCU1.P$14, SW1.P$7
- new net SW2: MCU1.P$8, SW1.P$6
- new net SW3: MCU1.P$7, SW1.P$5
- new net V3: CC1.P$2, IC1.P$5, MCU1.P$17
- new net V5: CC2.P$1, IC1.P$3, MCU1.P$27
- new net V5_MS: U$5.PIN20
- net CAN_H: now also CN1.P$5, IC1.P$7; no longer BOX10P-L1.P$5, U$2.P$7
- net CAN_L: now also CN1.P$6, IC1.P$6; no longer BOX10P-L1.P$6, U$2.P$6
- net CAN_RX: now also IC1.P$4, MCU1.P$13; no longer U$1.P$13, U$2.P$4
- net CAN_TX: now also IC1.P$1, MCU1.P$5; no longer U$1.P$5, U$2.P$1
- net GND: now also CC1.P$1, CC2.P$2, CN1.P$7, CN1.P$8, IC1.P$2, MCU1.P$29, MCU1.P$4, SW1.P$1, SW1.P$2, SW1.P$3, SW1.P$4, U$2.PIN2_S; no longer BOX10P-L1.P$7, BOX10P-L1.P$8, U$1.P$29, U$1.P$4
- net V12: now also CN1.P$1, CN1.P$2, MCU1.P$30; no longer BOX10P-L1.P$1, BOX10P-L1.P$2, U$1.P$30
Routing:
- net CAN_H: track 20.4 -> 0.00 mm
- net CAN_L: track 14.2 -> 0.00 mm
Other:
- board text added: "M2 washer"

Commit message: add dir
Connections:
- new net DIR: MCU1.P$9
Changed lines of the file:
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@@
 <wire x1="6.985" y1="36.82" x2="13.462" y2="6.985" width="0" layer="19" extent="1-1"/>
+</signal>
+<signal name="DIR" class="3">
+<contactref element="MCU1" pad="P$9"/>
 </signal>
 </signals>
