File: MotorSystemVS1/Motorsystem.sch (EAGLE design)
At the start: 3 parts

Commit message: continue
Parts:
- removed BOX10P-L1: BOX10PBOX10P-T, connectors:BOX10PBOX10P-T
- added CC1, CC2: 0.1u, capacitor:MLCC1608
- added CN1: BOX10P-T, connectors:BOX10P-T
- added IC1: MCP2562-SN, Microchip:MCP2562-SN
- added MCU1: NUCLEO-F303K8, Nucleo:NUCLEO-F303K8
- added SW1: KHS42SMD, switch:KHS42SMD
- added U$3: DF1B_L_4P, user:DF1B_L_4P
- added U$4, U$6, U$7, U$8: NP52N06SLG, user:NP52N06SLG
- added U$5: A3921, user:A3921
- added U$9: VL_4P, user:VL_4P
- U$1: value NUCLEO-F303K8 -> TLP2395; device Nucleo:NUCLEO-F303K8 -> user:TLP2395
- U$2: value MCP2561MCP2561-SN -> SOT23_NFET; device Microchip:MCP2561MCP2561-SN -> user:SOT23_NFET
Connections:
- new net CS: MCU1.PA0
- new net ENC_A: MCU1.PA5
- new net ENC_B: MCU1.PA1
- new net GND_MS: U$5.GND@1
- new net N$1: U$1.K, U$2.PIN3_D
- new net PWM: MCU1.PA8, U$2.PIN1_G
- new net PWM_MS: U$1.OUT, U$5.PWML
- new net SW0: MCU1.PB4, SW1.P$8
- new net SW1: MCU1.PB5, SW1.P$7
- new net SW2: MCU1.PB6, SW1.P$6
- new net SW3: MCU1.PB7, SW1.P$5
- new net V3: CC1.P$2, IC1.VIO, MCU1.+3V3
- new net V5: CC2.P$1, IC1.VDD, MCU1.+5V
- new net V5_MS: U$5.V5
- net CAN_H: now also CN1.P$5, IC1.CANH; no longer BOX10P-L1.P$5, U$2.CANH
- net CAN_L: now also CN1.P$6, IC1.CANL; no longer BOX10P-L1.P$6, U$2.CANL
- net CAN_RX: now also IC1.RXD, MCU1.PA11; no longer U$1.PA11, U$2.RXD
- net CAN_TX: now also IC1.TXD, MCU1.PA12; no longer U$1.PA12, U$2.TXD
- net GND: now also CC1.P$1, CC2.P$2, CN1.P$7, CN1.P$8, IC1.VSS, MCU1.GND@1, MCU1.GND@2, SW1.P$1, SW1.P$2, SW1.P$3, SW1.P$4, U$2.PIN2_S; no longer BOX10P-L1.P$7, BOX10P-L1.P$8, U$1.GND@1, U$1.GND@2
- net V12: now also CN1.P$1, CN1.P$2, MCU1.VIN; no longer BOX10P-L1.P$1, BOX10P-L1.P$2, U$1.VIN

Commit message: add dir
Connections:
- new net DIR: MCU1.PB1
Changed lines of the file:
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@@
+</segment>
+</net>
+<net name="DIR" class="3">
+<segment>
+<pinref part="MCU1" gate="G$1" pin="PB1"/>
+<wire x1="55.88" y1="45.72" x2="50.8" y2="45.72" width="0.1524" layer="91"/>
+<label x="50.8" y="45.72" size="1.778" layer="95" rot="R180" xref="yes"/>
 </segment>
 </net>
